File: Circuito/Circuito Robô/Placa.sch (EAGLE design)
At the start: 25 parts, among them IC1 LM317MBSTT3, M1 MOTOR10MM, M2 MOTOR10MM, U1 328P, X1 87438-03, X2 87438-03, X3 87438-03, X4 87438-03, X5 87438-03, X6 87438-03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

Commit message: Adiciona TB6612 e Trimpots
Parts:
- removed R2: 240Ω, resistor:R-US_M0805
- removed R3: 720Ω, resistor:R-US_M0805
- removed R4, R5: (no value), pot:TRIM_EU-3223W
- removed U$1: L298P013, SparkFun-IC-Special-Function:L298_BRIDGE_DRIVER
- added TB1: TB6612FNG, TB6612FNG:TB6612FNG
- added TM1, TM2, TM3, TM4: (no value), adafruit:TRIMPOT3386
Connections:
- removed net N$24: M2.+, R5.S
- new net N$22: TB1.PWMB, U1.PD5(T1)
- new net N$25: TM1.S, U1.PC3(ADC3)
- net GND: now also TB1.GND1, TM1.E, TM2.E, TM4.A; no longer R3.1, U$1.GND@1, U$1.GND@10, U$1.GND@11, U$1.GND@20, U$1.SENSE_A
- net N$10: now also TB1.PWMA, U1.PD3(INT1); no longer M1.-, U$1.OUT4, U$1.SENSE_B
- net N$11: now also TB1.STBY, U1.PB2(SS/OC1B); no longer R5.A, U$1.OUT1
- net N$12: now also TB1.BIN1, U1.PB3(MOSI/OC2); no longer M2.-, U$1.OUT2
- net N$13: now also TM3.A, TM4.S; no longer R2.1, R3.2
- net N$17: now also U1.PD2(INT0); no longer U1.PD5(T1)
- net N$21: now also TB1.BIN2, U1.PB4(MISO); no longer R4.A, U$1.OUT3
- net N$23: now also TM2.S, U1.PC4(ADC4/SDA); no longer M1.+, R4.S
- net N$4: now also TB1.AIN2; no longer U$1.IN1
- net N$5: now also TB1.AIN1, U1.PB1(OC1A); no longer U$1.IN2, U1.PB3(MOSI/OC2)
- net N$6: now also M1.+, TB1.A1; no longer U$1.IN3, U1.PB4(MISO)
- net N$7: now also M1.-, TB1.A2; no longer U$1.IN4, U1.PB5(SCK)
- net N$8: now also M2.-, TB1.B2; no longer U$1.ENA, U1.PB1(OC1A)
- net N$9: now also M2.+, TB1.B1; no longer U$1.ENB, U1.PB2(SS/OC1B)
- net VIN: now also TB1.VM; no longer U$1.VS
- net VO: now also TB1.VCC, TM1.A, TM2.A, TM3.S; no longer R2.2, U$1.VSS

Commit message: PCB com 125mm
Connections:
- net N$19: now also U1.PD5(T1); no longer U1.PD6(AIN0)
- net N$22: now also U1.PD6(AIN0); no longer U1.PD5(T1)
Other:
- moved on the sheet: X6-1, X6-2, X6-3
