File: Circuito/Circuito Robô/Placa.brd (EAGLE design)
At the start: 160 x 100 mm, 25 parts, among them IC1 LM317MBSTT3, M1 MOTOR10MM, M2 MOTOR10MM, U1 328P, X1 87438-03, X2 87438-03, X3 87438-03, X4 87438-03, X5 87438-03, X6 87438-03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

Commit message: Placa com 125mm
Parts:
- moved C2 206.2 mm to (143.5, 86.4)
- moved TB1 195.3 mm to (105.4, 64.8), turned to 270 degrees
- moved G1 183.4 mm to (144.8, 48.3)
- moved D2 179.1 mm to (135.9, 64.8), turned to 270 degrees
- moved D1 175.3 mm to (144.8, 64.8), turned to 90 degrees
- moved M1 170.0 mm to (113.0, 91.4)
- moved TM4 168.0 mm to (53.3, 27.9)
- moved M2 161.4 mm to (92.7, 85.1), turned to 180 degrees
- moved C1 156.0 mm to (134.6, 36.8)
- moved IC1 153.0 mm to (115.6, 31.8)
- moved TM1 151.9 mm to (35.6, 78.7)
- moved TM2 147.2 mm to (34.3, 54.6)
- moved C3 146.1 mm to (127.0, 55.9)
- moved TM3 144.5 mm to (34.3, 31.8)
- moved X5 124.5 mm to (64.8, 40.6), turned to 270 degrees
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Connections:
- net N$19: now also U1.11; no longer U1.12
- net N$22: now also U1.12; no longer U1.11
Routing:
- net VO: track 238.3 -> 454.8 mm, vias 2 -> 0
- net GND: track 207.5 -> 0.00 mm
- net N$18: track 13.1 -> 93.6 mm
- net N$25: track 0.00 -> 53.4 mm
- net N$13: track 84.2 -> 129.6 mm, vias 1 -> 0
- net N$10: track 0.00 -> 44.2 mm
- net N$23: track 0.00 -> 43.5 mm
- net N$17: track 54.3 -> 19.1 mm, vias 1 -> 0
- net N$3: track 52.5 -> 20.2 mm
- net N$2: track 31.7 -> 5.11 mm, vias 1 -> 0
- net N$1: track 31.0 -> 5.11 mm, vias 1 -> 0
- net N$7: track 0.00 -> 18.6 mm
- net N$20: track 22.4 -> 39.6 mm
- net N$9: track 0.00 -> 17.1 mm
- net N$6: track 0.00 -> 16.8 mm
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- added copper zone on layer 1, net GND
Other:
- board size 160 x 100 mm -> 125.7 x 70.8 mm
